File: patrick/patrick_v3_central/patrick_v3_central.kicad_pcb (KiCad board)
At the start: 2 copper layers, 36 x 36 mm, 55 parts, among them J1 Conn_02x05_Counter_Clockwise, J10 61300311121, J2 Conn_02x05_Counter_Clockwise, J3 Conn_02x05_Counter_Clockwise, J4 Conn_02x05_Counter_Clockwise, J5 Conn_02x05_Counter_Clockwise, J7 61300211121, J9 61300211121, U1 TCA9548APWR, U3 BL652-SA-01

Commit message: modified patrick boards
Parts:
- removed RP1, RP10, RP11, RP12, RP13, RP14, RP15, RP16, RP17, RP18, RP19, RP2, RP20, RP3, RP4, RP5, RP6, RP7, RP8, RP9, RS1, RS10, RS11, RS12, RS13, RS14, RS15, RS16, RS17, RS18, RS19, RS2, RS20, RS3, RS4, RS5, RS6, RS7, RS8, RS9: , Resistor_SMD:R_0402_1005Metric
- removed U1: TCA9548APWR, TCA9548A:SOP65P640X120-24N
- J1, J2, J3, J4, J5: footprint MolexPicoClasp:Molex_Pico-Clasp_501331-1007_1x10-1MP_P1.00mm_Vertical -> Connector_PinHeader_1.00mm:PinHeader_1x10_P1.00mm_Vertical
- moved R2 12.1 mm to (118.3, 118.8), turned to 0 degrees
- moved R1 6.66 mm to (112.6, 122.8)
- moved J4 5.45 mm to (102.3, 118.5), turned to 225 degrees
- moved J1 4.74 mm to (121.5, 104.8), turned to 0 degrees
- moved J2 4.40 mm to (110.7, 95.9), turned to 60 degrees
- moved J3 3.32 mm to (96.0, 105.0), turned to 135 degrees
- moved J5 1.87 mm to (114.4, 120.6), turned to 285 degrees
Connections:
- J1 pad 5: /SMA12_PWR -> /SMA12_SIG
- J1 pad 6: /SMA11_PWR -> /SMA11_SIG
- J1 pad 7: /SMA10_PWR -> /SMA10_SIG
- J1 pad 8: /SMA9_PWR -> /SMA9_SIG
- J2 pad 5: /SMA16_PWR -> /SMA16_SIG
- J2 pad 6: /SMA15_PWR -> /SMA15_SIG
- J2 pad 7: /SMA14_PWR -> /SMA14_SIG
- J2 pad 8: /SMA13_PWR -> /SMA13_SIG
- J3 pad 5: /SMA20_PWR -> /SMA20_SIG
- J3 pad 6: /SMA19_PWR -> /SMA19_SIG
- J3 pad 7: /SMA18_PWR -> /SMA18_SIG
- J3 pad 8: /SMA17_PWR -> /SMA17_SIG
- J4 pad 5: /SMA4_PWR -> /SMA4_SIG
- J4 pad 6: /SMA3_PWR -> /SMA3_SIG
- J4 pad 7: /SMA2_PWR -> /SMA2_SIG
- J4 pad 8: /SMA1_PWR -> /SMA1_SIG
- J5 pad 5: /SMA8_PWR -> /SMA8_SIG
- J5 pad 6: /SMA7_PWR -> /SMA7_SIG
- J5 pad 7: /SMA6_PWR -> /SMA6_SIG
- J5 pad 8: /SMA5_PWR -> /SMA5_SIG
- U3 pad 33: Net-(U3-Pad33) -> /SMA20_SIG
- U3 pad 34: /SMA20_SIG -> /SMA19_SIG
- U3 pad 35: /SMA19_SIG -> Net-(U3-Pad35)
Routing:
- net GND: track 263.1 -> 189.1 mm, vias 18 -> 8
- net /SMA17_SIG: track 9.13 -> 20.7 mm
- net /+3V: track 132.9 -> 122.5 mm, vias 5 -> 1
- net /SMA9_SIG: track 2.15 -> 9.56 mm
- net /SMA16_PWR: track 7.39 -> 0.00 mm
- net /SMA17_PWR: track 7.03 -> 0.00 mm
- net /SMA13_PWR: track 6.63 -> 0.00 mm
- net /SMA5_PWR: track 6.45 -> 0.00 mm
- net /SMA9_PWR: track 6.40 -> 0.00 mm
- net /SMA4_PWR: track 6.37 -> 0.00 mm
- net /SMA10_SIG: track 3.06 -> 9.42 mm
- net /SMA1_PWR: track 6.31 -> 0.00 mm
- net /SMA8_PWR: track 6.07 -> 0.00 mm
- net /SMA5_SIG: track 1.69 -> 7.50 mm
- net /SMA10_PWR: track 5.68 -> 0.00 mm
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
Commit message: switched connectors
Parts:
- J1, J2, J3, J4, J5: footprint Connector_PinHeader_1.00mm:PinHeader_1x10_P1.00mm_Vertical -> Connector_PinHeader_2.00mm:PinHeader_2x05_P2.00mm_Vertical
- moved J4 9.54 mm to (93.7, 122.7), turned to 210 degrees
- moved J1 8.27 mm to (129.3, 107.4), turned to 354 degrees
- moved J5 7.93 mm to (117.1, 128.1), turned to 282 degrees
- moved J3 7.41 mm to (91.7, 99.0), turned to 138 degrees
- moved J2 6.95 mm to (113.6, 89.6), turned to 66 degrees
Connections:
- J1 pad 2: /SCL -> /SDA
- J1 pad 3: /SDA -> /SMA12_SIG
- J1 pad 4: Net-(J1-Pad4) -> /SCL
- J1 pad 5: /SMA12_SIG -> /SMA11_SIG
- J1 pad 6: /SMA11_SIG -> Net-(J1-Pad6)
- J2 pad 2: /SCL -> /SDA
- J2 pad 3: /SDA -> /SMA16_SIG
- J2 pad 4: Net-(J2-Pad4) -> /SCL
- J2 pad 5: /SMA16_SIG -> /SMA15_SIG
- J2 pad 6: /SMA15_SIG -> Net-(J2-Pad6)
- J3 pad 2: /SCL -> /SDA
- J3 pad 3: /SDA -> /SMA20_SIG
- J3 pad 4: Net-(J3-Pad4) -> /SCL
- J3 pad 5: /SMA20_SIG -> /SMA19_SIG
- J3 pad 6: /SMA19_SIG -> Net-(J3-Pad6)
- J4 pad 2: /SCL -> /SDA
- J4 pad 3: /SDA -> /SMA4_SIG
- J4 pad 4: Net-(J4-Pad4) -> /SCL
- J4 pad 5: /SMA4_SIG -> /SMA3_SIG
- J4 pad 6: /SMA3_SIG -> Net-(J4-Pad6)
- J5 pad 2: /SCL -> /SDA
- J5 pad 3: /SDA -> /SMA8_SIG
- J5 pad 4: Net-(J5-Pad4) -> /SCL
- J5 pad 5: /SMA8_SIG -> /SMA7_SIG
- J5 pad 6: /SMA7_SIG -> Net-(J5-Pad6)
Routing:
- net /SCL: track 91.6 -> 187.9 mm, vias 1 -> 7
- net /SDA: track 78.2 -> 148.1 mm, vias 5 -> 7
- net +8V: track 139.1 -> 188.5 mm, vias 5 -> 1
- net /+3V: track 122.5 -> 149.6 mm, vias 1 -> 5
- net /SMA9_SIG: track 9.56 -> 27.7 mm
- net /SMA5_SIG: track 7.50 -> 24.9 mm
- net /SMA13_SIG: track 13.9 -> 30.4 mm
- net /SMA1_SIG: track 7.23 -> 23.6 mm
- net /SMA17_SIG: track 20.7 -> 32.9 mm
- net /SMA19_SIG: track 13.4 -> 24.9 mm
- net /SMA20_SIG: track 13.0 -> 24.0 mm
- net /SMA4_SIG: track 5.05 -> 14.0 mm
- net /SMA3_SIG: track 5.78 -> 14.6 mm
- net /SMA8_SIG: track 6.89 -> 15.6 mm
- net /SMA2_SIG: track 6.94 -> 15.7 mm
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Other:
- board size 36 x 36 mm -> 49.5 x 50 mm
