File: patrick/patrick_0.5/patrick_0_5.kicad_pcb (KiCad board)
At the start: 2 copper layers, 29 x 29 mm, 86 parts, among them J10 61300311121, J7 61300211121, J9 61300211121, P1 CONN_01, P10 CONN_01, P11 CONN_01, P12 CONN_01, P13 CONN_01, P14 CONN_01, P15 CONN_01, P16 CONN_01, P17 CONN_01, P18 CONN_01, P19 CONN_01, P2 CONN_01, P20 CONN_01, P3 CONN_01, P4 CONN_01, P5 CONN_01, P6 CONN_01, P7 CONN_01, P8 CONN_01, P9 CONN_01, Q1 MOSFET-NREFLOW, Q10 MOSFET-NREFLOW, Q11 MOSFET-NREFLOW, Q12 MOSFET-NREFLOW, Q13 MOSFET-NREFLOW, Q14 MOSFET-NREFLOW, Q15 MOSFET-NREFLOW, Q16 MOSFET-NREFLOW, Q17 MOSFET-NREFLOW, Q18 MOSFET-NREFLOW, Q19 MOSFET-NREFLOW, Q2 MOSFET-NREFLOW, Q20 MOSFET-NREFLOW, Q3 MOSFET-NREFLOW, Q4 MOSFET-NREFLOW, Q5 MOSFET-NREFLOW, Q6 MOSFET-NREFLOW, Q7 MOSFET-NREFLOW, Q8 MOSFET-NREFLOW, Q9 MOSFET-NREFLOW, U3 BL652-SA-01

Commit message: adding patrick boards
Parts:
- J10: footprint Connector_PinHeader_1.27mm:PinHeader_1x02_P1.27mm_Vertical -> Connector_PinHeader_1.27mm:PinHeader_1x03_P1.27mm_Vertical
- moved J10 17.4 mm to (117.7, 110.7)
- moved J9 17.3 mm to (100.3, 110.4)
Connections:
- J10 pad 1: /+3V -> /RESET
- J10 pad 2: GND -> /SWDCLK
- J9 pad 1: /SWDCLK -> /+3V
- J9 pad 2: /SWDIO -> GND
- U3 pad 30: Net-(U3-Pad30) -> /SMA4_SIG
- U3 pad 31: Net-(U3-Pad31) -> /SMA3_SIG
- U3 pad 32: /SMA4_SIG -> /SMA2_SIG
- U3 pad 33: /SMA3_SIG -> /SMA1_SIG
- U3 pad 34: /SMA2_SIG -> /SMA20_SIG
- U3 pad 35: /SMA1_SIG -> /SMA19_SIG
- U3 pad 36: /SMA20_SIG -> Net-(U3-Pad36)
- U3 pad 37: /SMA19_SIG -> Net-(U3-Pad37)
Routing:
- net /RESET: track 0.00 -> 4.94 mm
- net /SMA20_SIG: track 4.27 -> 8.14 mm
- net /SMA18_SIG: track 5.31 -> 7.82 mm
- net /SMA4_SIG: track 4.41 -> 6.49 mm
- net /SMA2_SIG: track 3.02 -> 4.75 mm
- net GND: track 194.0 -> 195.0 mm
- net /SMA19_SIG: track 4.63 -> 5.63 mm
- net /SMA3_SIG: track 3.33 -> 4.27 mm
- net /SMA1_SIG: track 3.64 -> 4.53 mm
