File: patrick/patrick_v4/patrick_v3.kicad_pcb (KiCad board)
At the start: 2 copper layers, 26.6 x 30.1 mm, 22 parts, among them J1 Conn_02x05_Counter_Clockwise, J10 Conn_01x01, J2 Conn_01x01, J3 Conn_01x01, J4 Conn_01x01, J5 Conn_01x01, J6 Conn_01x01, J7 Conn_01x01, J8 Conn_01x01, J9 Conn_01x01, Q1 Q_NMOS_GSD, Q2 Q_NMOS_GSD, Q3 Q_NMOS_GSD, Q4 Q_NMOS_GSD

Commit message: added a few updated patrick designs
Other:
- board size 26.6 x 30.1 mm -> 21 x 13 mm
