File: patrick/patrick_v5_central_3leg_tethered/patrick_v3_central.kicad_pcb (KiCad board)
At the start: 2 copper layers, 47.6 x 51.7 mm, 11 parts, among them J1 Conn_02x05_Counter_Clockwise, J2 Conn_01x31, J4 Conn_02x05_Counter_Clockwise, J5 Conn_02x05_Counter_Clockwise, U1 ZLDO1117G33TA, U2 ICM-20948, U4 MCP1703T-1802E_CB

Commit message: thethered robot boards and TLC breackout
Parts:
- removed C1, C2: C-USC0402, Capacitor_SMD:C_0402_1005Metric_Pad0.74x0.62mm_HandSolder
- removed U1: ZLDO1117G33TA, ZLDO1117G33TA:SOT230P700X180-4N
- moved U2 7.76 mm to (103.9, 121.0), turned to 270 degrees
- moved U4 3.05 mm to (112.2, 120.4)
- moved C3 2.52 mm to (107.4, 121.2), turned to 270 degrees
- moved C4 1.08 mm to (108.7, 121.2), turned to 270 degrees
Connections:
- J2 pad 11: Net-(J2-Pad11) -> /SCL
- J2 pad 12: Net-(J2-Pad12) -> /SMA10_SIG
- J2 pad 13: /SMA9_SIG -> /SMA8_SIG
- J2 pad 14: /SMA1_SIG -> Net-(J2-Pad14)
- J2 pad 17: Net-(J2-Pad17) -> /SDA
- J2 pad 18: Net-(J2-Pad18) -> /SMA7_SIG
- J2 pad 19: /SMA2_SIG -> Net-(J2-Pad19)
- J2 pad 23: Net-(J2-Pad23) -> /+3V
- J2 pad 24: /SMA8_SIG -> /SMA6_SIG
- J2 pad 25: /SMA3_SIG -> Net-(J2-Pad25)
- J2 pad 26: /SMA4_SIG -> Net-(J2-Pad26)
- J2 pad 27: Net-(J2-Pad27) -> /SMA2_SIG
- J2 pad 28: /SMA6_SIG -> /SMA4_SIG
- J2 pad 29: /SMA7_SIG -> /SMA5_SIG
- J2 pad 30: Net-(J2-Pad30) -> /SMA1_SIG
- J2 pad 31: /SMA5_SIG -> /SMA3_SIG
- J2 pad 7: /SMA10_SIG -> /SMA9_SIG
Routing:
- net /SCL: track 0.00 -> 209.2 mm, vias 0 -> 5
- net /SDA: track 0.00 -> 176.7 mm, vias 0 -> 2
- net +8V: track 23.8 -> 135.7 mm, vias 0 -> 3
- net /+3V: track 0.00 -> 87.9 mm, vias 0 -> 3
- net GND: track 92.5 -> 173.5 mm
- net Net-(C4-Pad1): track 0.00 -> 12.3 mm
- net Net-(U2-Pad1): track 0.00 -> 11.2 mm
- net /SMA2_SIG: track 15.7 -> 25.3 mm
- net /SMA4_SIG: track 19.7 -> 27.5 mm
- net /SMA3_SIG: track 16.1 -> 23.5 mm
- net /SMA1_SIG: track 18.5 -> 23.7 mm
- net /SMA8_SIG: track 17.9 -> 20.9 mm
- net /SMA5_SIG: track 20.6 -> 17.6 mm
- net /SMA6_SIG: track 20.6 -> 17.8 mm
- net /SMA9_SIG: track 20.4 -> 17.7 mm
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Other:
- net class Default: clearance 0.1 -> 0.15
- rule trace_clearance: 0.1 -> 0.15
