File: patrick/patrick_limb_adapter/patrick_limb_adapter.kicad_pcb (KiCad board)
At the start: 2 copper layers, 19.4 x 14.2 mm, 3 parts, among them J1 Conn_01x05, J2 Conn_02x05_Counter_Clockwise, J3 Conn_01x05

Commit message: v5 circuit
Connections:
- net Net-(J1-Pad1) renamed /SMA1
- net Net-(J1-Pad2) renamed /SDA
- net Net-(J1-Pad5) renamed /GND
- net Net-(J2-Pad10) renamed /12V
- net Net-(J2-Pad6) renamed /SCL
- net Net-(J2-Pad7) renamed /SMA4
- net Net-(J2-Pad8) renamed /SMA3
- net Net-(J2-Pad9) renamed /3.3V
- J1 pad 3: Net-(J1-Pad3) -> /SMA2
- J1 pad 4: Net-(J1-Pad4) -> /SMA2
- J2 pad 2: Net-(J1-Pad4) -> /SMA2
- J2 pad 3: Net-(J1-Pad3) -> /SMA2
Routing:
- net /SMA2: track 0.00 -> 29.2 mm
- net Net-(J1-Pad3): track 19.8 -> 0.00 mm
- net Net-(J1-Pad4): track 9.36 -> 0.00 mm
