File: patrick/patrick_limb_adapter/patrick_limb_adapter.sch (KiCad schematic (older format))
At the start: 3 parts, among them J1 Conn_01x05, J2 Conn_02x05_Counter_Clockwise, J3 Conn_01x05

Commit message: v5 circuit
Connections:
- net GND: now reaches J1.5 (Pin_5), J2.1 (Pin_1)
- net 12V: now reaches J2.10 (Pin_10), J3.1 (Pin_1)
- net SMA2: now reaches J1.4 (Pin_4), J2.2 (Pin_2)
- net SMA2: now also J1.3 (Pin_3), J2.3 (Pin_3)
- net SDA: now reaches J1.2 (Pin_2), J2.4 (Pin_4)
- net SMA1: now reaches J1.1 (Pin_1), J2.5 (Pin_5)
- net SCL: now reaches J2.6 (Pin_6), J3.5 (Pin_5)
- net SMA4: now reaches J2.7 (Pin_7), J3.4 (Pin_4)
- net SMA3: now reaches J2.8 (Pin_8), J3.3 (Pin_3)
- net 3.3V: now reaches J2.9 (Pin_9), J3.2 (Pin_2)
Changed lines of the file:
@@
 	-1   0    0    1
 $EndComp
+Text Label 5900 3450 0    50   ~ 0
+SDA
+Text Label 6400 3550 0    50   ~ 0
+SCL
+Text Label 6400 3250 0    50   ~ 0
+3.3V
+Text Label 5900 3150 0    50   ~ 0
+GND
+Text Label 6400 3150 0    50   ~ 0
+12V
+Text Label 5900 3550 0    50   ~ 0
+SMA1
+Text Label 5900 3250 0    50   ~ 0
+SMA2
+Text Label 5900 3350 0    50   ~ 0
+SMA2
+Text Label 6400 3350 0    50   ~ 0
+SMA3
+Text Label 6400 3450 0    50   ~ 0
+SMA4
 $EndSCHEMATC
