File: patrick/patrick_v5_untethered_central/patrick_v3_central.sch (KiCad schematic (older format))
At the start: 24 parts, among them IC1 IS32FL3237-TQLA3, J1 Conn_02x05_Counter_Clockwise, J10 61300311121, J2 Conn_02x05_Counter_Clockwise, J3 Conn_02x05_Counter_Clockwise, J4 Conn_02x05_Counter_Clockwise, J5 Conn_02x05_Counter_Clockwise, J6 DM3CS-SF, J7 61300211121, J8 Conn_01x03, U1 ICM-20948, U2 MCP1702T-1802E_CB, U3 BL652-SA-01

Commit message: imu change
Parts:
- added Q1, Q2, Q3: RUE002N02TL, RUE002N02TL:TRANS_RUE002N02TL, symbol RUE002N02TL:RUE002N02TL
- added R5, R6, R7: (no value), Resistor_SMD:R_0402_1005Metric, symbol patrick_0.5-eagle-import:RESISTOR0402
Connections:
- net labels added: INT, INT_VIN, SCL_VIN, SDA_VIN
- wire segments 127 -> 136
Other:
- moved on the sheet: C1, C2, C3, C4, C5, C6, IC1, J1, J10, J2, J3, J4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

Commit message: LED switcher useless
Parts:
- J6: symbol DM3CS-SF:DM3CS-SF -> patrick_v3_central-rescue:DM3CS-SF-DM3CS-SF
- Q1, Q2, Q3: symbol RUE002N02TL:RUE002N02TL -> patrick_v3_central-rescue:RUE002N02TL-RUE002N02TL
- U1: symbol ICM-20948:ICM-20948 -> patrick_v3_central-rescue:ICM-20948-ICM-20948
- U2: symbol 2022-05-16_19-05-33:MCP1702T-1802E_CB -> patrick_v3_central-rescue:MCP1702T-1802E_CB-2022-05-16_19-05-33
Changed lines of the file:
@@
 	1    0    0    -1
 $EndComp
+Text Label 3650 4900 1    50   ~ 0
+SCL
 Text Label 3750 4900 1    50   ~ 0
-SCL
-Text Label 3650 4900 1    50   ~ 0
 SDA
 Wire Wire Line
+	3750 4450 3750 4950
+Wire Wire Line
 	3650 4450 3650 4950
-Wire Wire Line
-	3750 4450 3750 4950
 Text Label 3050 6450 2    70   ~ 0
 SMA20_SIG
@@
 	5700 5000 5700 4750
 $Comp
-L 2022-05-16_19-05-33:MCP1702T-1802E_CB U2
+L patrick_v3_central-rescue:MCP1702T-1802E_CB-2022-05-16_19-05-33 U2
 U 1 1 629E7A37
 P 13100 7200
@@
 $EndComp
 $Comp
-L ICM-20948:ICM-20948 U1
+L patrick_v3_central-rescue:ICM-20948-ICM-20948 U1
 U 1 1 629EFB4A
 P 11900 5050
@@
 	9250 4900 10550 4900
 $Comp
-L DM3CS-SF:DM3CS-SF J6
+L patrick_v3_central-rescue:DM3CS-SF-DM3CS-SF J6
 U 1 1 6283BBA7
 P 10800 2300
@@
 	4150 4900 4150 4950
 $Comp
-L RUE002N02TL:RUE002N02TL Q1
+L patrick_v3_central-rescue:RUE002N02TL-RUE002N02TL Q1
 U 1 1 629F26AC
 P 13700 5750
@@
 	15250 5000 15250 5500
 $Comp
-L RUE002N02TL:RUE002N02TL Q2
+L patrick_v3_central-rescue:RUE002N02TL-RUE002N02TL Q2
 U 1 1 62A179F5
 P 15150 5800
@@
 	16550 5000 16550 5500
 $Comp
-L RUE002N02TL:RUE002N02TL Q3
+L patrick_v3_central-rescue:RUE002N02TL-RUE002N02TL Q3
 U 1 1 62A6627A
 P 16450 5800
