File: patrick/patrick_v6_central_3leg/patrick_v3_central.sch (KiCad schematic (older format))
At the start: 27 parts, among them J1 Conn_02x05_Counter_Clockwise, J10 61300311121, J4 Conn_02x05_Counter_Clockwise, J5 Conn_02x05_Counter_Clockwise, J7 61300211121, J9 61300211121, Q1 RUE002N02TL, Q2 RUE002N02TL, Q3 RUE002N02TL, U1 MPM3610GQV-Z, U2 ICM-20948, U3 BL652-SA-01, U4 MCP1703T-1802E_CB

Commit message: separate gnd
Parts:
- added 1: V_REG_SPX3819-SOT23-5, Package_TO_SOT_SMD:SOT-23-5, symbol patrick_0.5-eagle-import:V_REG_SPX3819-SOT23-5
- added C7: CP1_Small, Capacitor_THT:CP_Radial_D4.0mm_P2.00mm, symbol Device:CP1_Small
- added J2: Conn_01x02, Connector_PinSocket_2.00mm:PinSocket_1x02_P2.00mm_Vertical, symbol Connector_Generic:Conn_01x02
- added JP1, JP2: Jumper_NO_Small, Jumper:SolderJumper-2_P1.3mm_Open_RoundedPad1.0x1.5mm, symbol Device:Jumper_NO_Small
- U4: symbol MCP1703T-1802E_CB:MCP1703T-1802E_CB -> patrick_v3_central-rescue:MCP1703T-1802E_CB-MCP1703T-1802E_CB
Connections:
- net labels added: GND2
- wire segments 112 -> 116
